File: kicadFiles/keebsPCB.kicad_pcb (KiCad board)
At the start: 2 copper layers, 107 x 16 mm, 57 parts, among them SW1 ESC, SW10 9, SW11 0, SW12 -_, SW13 =+, SW14 BCKSPC_200, SW15 TAB_150, SW16 Q, SW17 W, SW18 E, SW19 R, SW2 1, SW20 T, SW21 Y, SW22 U, SW23 I, SW24 O, SW25 P, SW26 [{, SW29 CAPSLOCK_175, SW3 2, SW30 A, SW31 S, SW32 D, SW33 F, SW34 G, SW35 H, SW36 J, SW37 K, SW38 L, SW39 ;:, SW4 3, SW40 ', SW41 ENTER_ISO, SW42 LSHIFT_125, SW5 4, SW53 RSHIFT_275, SW54 LCTRL_125, SW55 LGUI_125, SW56 LALT_125, SW57 SPACE_625, SW58 RALT_125, SW59 RGUI_125, SW6 5, SW60 FN_125, SW61 RCTRL_125, SW7 6, SW8 7, SW9 8

Commit message: reset
Parts:
- removed HOLE (x8): H**, acheron_MountingHoles:MountingHole_2.5x5.0mm
- removed SW61: RCTRL_125, muente_plate:MX100
- added CB1: 1uF, Capacitor_SMD:C_0402_1005Metric, F.Cu at (318.1, 138.1)
- added CB2: 10n, Capacitor_SMD:C_0402_1005Metric, F.Cu at (319.3, 138.1)
- added CB3: 100n, Capacitor_SMD:C_0402_1005Metric, F.Cu at (333.3, 133.8)
- added CB4: 4.7uF, Capacitor_SMD:C_0402_1005Metric, F.Cu at (333.3, 132.6)
- added CB5: 100n, Capacitor_SMD:C_0402_1005Metric, F.Cu at (329.4, 143.4)
- added CB6: 4.7uF, Capacitor_SMD:C_0402_1005Metric, F.Cu at (330.6, 143.4)
- added CB7: 100nF, Capacitor_SMD:C_0402_1005Metric, F.Cu at (320.2, 133.7)
- added CB8: 100n, Capacitor_SMD:C_0402_1005Metric, F.Cu at (321.2, 132.4)
- added CRST1: 10u, Capacitor_SMD:C_0805_2012Metric_Pad1.15x1.40mm_HandSolder, F.Cu at (279.7, 155.1)
- added CRST2: 4.7n, Capacitor_SMD:C_0805_2012Metric_Pad1.15x1.40mm_HandSolder, F.Cu at (290.9, 156.2)
- added CSH1: 4.7nF, Capacitor_SMD:C_0805_2012Metric, F.Cu at (328.0, 102.3)
- added CSI1: 10u, Capacitor_SMD:C_0805_2012Metric_Pad1.15x1.40mm_HandSolder, F.Cu at (303.7, 116.6)
- added CSO1: 1u, Capacitor_SMD:C_0805_2012Metric_Pad1.15x1.40mm_HandSolder, F.Cu at (297.7, 115.6)
- added CUSB1: 100n, Capacitor_SMD:C_0402_1005Metric, F.Cu at (332.3, 117.0)
- added D1: 1N4148, acheron_Components:D_SOD-123, F.Cu at (318.0, 115.7)
- added D10: 1N4148, acheron_Components:D_SOD-123, F.Cu at (184.7, 110.9)
- added D11: 1N4148, acheron_Components:D_SOD-123, F.Cu at (165.6, 110.9)
- added D12: 1N4148, acheron_Components:D_SOD-123, F.Cu at (146.6, 113.3)
- added D13: 1N4148, acheron_Components:D_SOD-123, F.Cu at (127.5, 110.9)
- added D14: 1N4148, acheron_Components:D_SOD-123, F.Cu at (98.9, 110.9)
- added D15: 1N4148, acheron_Components:D_SOD-123, F.Cu at (351.4, 120.4)
- added D16: 1N4148, acheron_Components:D_SOD-123, F.Cu at (327.5, 120.4)
- added D17: 1N4148, acheron_Components:D_SOD-123, F.Cu at (308.5, 120.4)
- added D18: 1N4148, acheron_Components:D_SOD-123, F.Cu at (289.4, 120.4)
- added D19: 1N4148, acheron_Components:D_SOD-123, F.Cu at (270.4, 120.4)
- added D2: 1N4148, acheron_Components:D_SOD-123, F.Cu at (320.4, 106.1)
- added D20: 1N4148, acheron_Components:D_SOD-123, F.Cu at (251.3, 120.4)
- added D21: 1N4148, acheron_Components:D_SOD-123, F.Cu at (232.3, 120.4)
- added D22: 1N4148, acheron_Components:D_SOD-123, F.Cu at (213.2, 120.4)
- added D23: 1N4148, acheron_Components:D_SOD-123, F.Cu at (194.2, 120.4)
- added D24: 1N4148, acheron_Components:D_SOD-123, F.Cu at (175.1, 120.4)
- added D25: 1N4148, acheron_Components:D_SOD-123, F.Cu at (156.1, 120.4)
- added D26: 1N4148, acheron_Components:D_SOD-123, F.Cu at (137.0, 120.4)
- added D27: 1N4148, acheron_Components:D_SOD-123, F.Cu at (118.0, 120.4)
- added D28: 1N4148, acheron_Components:D_SOD-123, F.Cu at (96.6, 120.4)
- added D29: 1N4148, acheron_Components:D_SOD-123, F.Cu at (339.4, 151.4)
- added D3: 1N4148, acheron_Components:D_SOD-123, F.Cu at (315.6, 110.9)
- added D30: 1N4148, acheron_Components:D_SOD-123, F.Cu at (320.4, 151.4)
- added D31: 1N4148, acheron_Components:D_SOD-123, F.Cu at (301.3, 151.4)
- added D32: 1N4148, acheron_Components:D_SOD-123, F.Cu at (282.3, 151.4)
- added D33: 1N4148, acheron_Components:D_SOD-123, F.Cu at (263.2, 151.4)
- added D34: 1N4148, acheron_Components:D_SOD-123, F.Cu at (244.2, 151.4)
- added D35: 1N4148, acheron_Components:D_SOD-123, F.Cu at (225.1, 151.4)
- added D36: 1N4148, acheron_Components:D_SOD-123, F.Cu at (206.1, 151.4)
- added D37: 1N4148, acheron_Components:D_SOD-123, F.Cu at (187.0, 151.4)
- added D38: 1N4148, acheron_Components:D_SOD-123, F.Cu at (168.0, 151.4)
- added D39: 1N4148, acheron_Components:D_SOD-123, F.Cu at (148.9, 151.4)
- added D4: 1N4148, acheron_Components:D_SOD-123, F.Cu at (298.3, 101.8)
- added D40: 1N4148, acheron_Components:D_SOD-123, F.Cu at (129.9, 151.4)
- added D41: 1N4148, acheron_Components:D_SOD-123, F.Cu at (98.9, 151.4)
- added D42: 1N4148, acheron_Components:D_SOD-123, F.Cu at (344.2, 168.0)
- added D43: 1N4148, acheron_Components:D_SOD-123, F.Cu at (313.3, 168.0)
- added D44: 1N4148, acheron_Components:D_SOD-123, F.Cu at (294.2, 168.0)
- added D45: 1N4148, acheron_Components:D_SOD-123, F.Cu at (275.2, 168.0)
- added D46: 1N4148, acheron_Components:D_SOD-123, F.Cu at (256.1, 168.0)
- added D47: 1N4148, acheron_Components:D_SOD-123, F.Cu at (237.1, 168.0)
- added D48: 1N4148, acheron_Components:D_SOD-123, F.Cu at (218.0, 168.0)
- added D49: 1N4148, acheron_Components:D_SOD-123, F.Cu at (199.0, 168.0)
- added D5: 1N4148, acheron_Components:D_SOD-123, F.Cu at (279.9, 113.3)
- added D50: 1N4148, acheron_Components:D_SOD-123, F.Cu at (179.9, 168.0)
- added D51: 1N4148, acheron_Components:D_SOD-123, F.Cu at (160.9, 168.0)
- added D52: 1N4148, acheron_Components:D_SOD-123, F.Cu at (141.8, 168.0)
- added D53: 1N4148, acheron_Components:D_SOD-123, F.Cu at (106.1, 168.0)
- added D54: 1N4148, acheron_Components:D_SOD-123, F.Cu at (349.0, 189.5)
- added D55: 1N4148, acheron_Components:D_SOD-123, F.Cu at (325.2, 189.5)
- added D56: 1N4148, acheron_Components:D_SOD-123, F.Cu at (301.3, 189.5)
- added D57: 1N4148, acheron_Components:D_SOD-123, F.Cu at (220.4, 189.5)
- added D58: 1N4148, acheron_Components:D_SOD-123, F.Cu at (139.4, 189.5)
- added D59: 1N4148, acheron_Components:D_SOD-123, F.Cu at (115.6, 189.5)
- added D6: 1N4148, acheron_Components:D_SOD-123, F.Cu at (260.9, 110.9)
- added D60: 1N4148, acheron_Components:D_SOD-123, F.Cu at (90.3, 189.5)
- added D7: 1N4148, acheron_Components:D_SOD-123, F.Cu at (241.8, 110.9)
- added D8: 1N4148, acheron_Components:D_SOD-123, F.Cu at (222.8, 110.9)
- added D9: 1N4148, acheron_Components:D_SOD-123, F.Cu at (203.7, 110.9)
- added DF1: RB060M-60TR, acheron_Components:D_SOD-123, F.Cu at (306.2, 115.6)
- added DRST1: 1N4148, acheron_Components:D_SOD-123, F.Cu at (275.0, 155.1)
- added DS1: 1N4148, acheron_Components:D_SOD-123, F.Cu at (300.7, 112.1)
- added F1: Polyfuse, acheron_Components:Fuse_1812_4532, F.Cu at (310.9, 115.5)
- added H1: Half Side Hole, acheron_MountingHoles:halfSideHole, B.Cu at (354.7, 156.1)
- added H10: Oval Mounting Hole, acheron_MountingHoles:MoutingHole_Oval_BackOnly_7mm_5.0x2.5mm, B.Cu at (146.6, 108.5)
- added H2: Mounting Hole, acheron_MountingHoles:MoutingHole_Oval_7mm_5.0x2.5mm, B.Cu at (331.1, 127.6)
- added H3: Oval Mounting Hole, acheron_MountingHoles:MoutingHole_Oval_BackOnly_7mm_5.0x2.5mm, B.Cu at (227.5, 146.6)
- added H4: Oval Mounting Hole, acheron_MountingHoles:MoutingHole_Oval_7mm_5.0x2.5mm, B.Cu at (165.3, 184.5)
- added H5: Oval Mounting Hole, acheron_MountingHoles:MoutingHole_Oval_BackOnly_7mm_5.0x2.5mm, B.Cu at (95.7, 127.6)
- added H6: Half Side Hole, acheron_MountingHoles:halfSideHole, B.Cu at (71.7, 156.1)
- added H7: Oval Mounting Hole, acheron_MountingHoles:MoutingHole_Oval_7mm_5.0x2.5mm, F.Cu at (331.7, 184.5)
- added H8: Oval Mounting Hole, acheron_MountingHoles:MoutingHole_Oval_BackOnly_7mm_5.0x2.5mm, B.Cu at (279.9, 108.5)
- added H9: Oval Mounting Hole, acheron_MountingHoles:MoutingHole_Oval_7mm_5.0x2.5mm, F.Cu at (96.3, 188.1)
- added J1: TYPE-C-31-M12_13, acheron_Connectors:TYPE-C-31-M-12, F.Cu at (337.1, 106.7)
- added J2: Conn_ARM_JTAG_SWD_10, acheron_Connectors:Conn_ARM_JTAG_SWD_10, F.Cu at (279.9, 184.7)
- added J3: Conn_01x14, acheron_Connectors:PinHeader_1x7_P2.54mm_Vertical, F.Cu at (352.4, 136.5)
- added J4: Conn_01x14, acheron_Connectors:PinHeader_1x8_P2.54mm_Vertical, F.Cu at (352.4, 166.4)
- added L1: Keebs Logo, keebsLogo:keebsLogo, B.Cu at (244.2, 183.9)
- added L2: OSHLogo, oshLogo:osh-logo, F.Cu at (277.1, 134.7)
- added L3: Keebs Label, keebsLogo:keebsLabel, F.Cu at (186.6, 182.4)
- added L4: Keebs Label Mask, keebsLogo:keebsLabelMask, F.Cu at (186.6, 182.4)
- added QRST1: DTC123J, Package_TO_SOT_SMD:SOT-23, F.Cu at (287.9, 156.2)
- added RCC1: 5.1k, Resistor_SMD:R_0402_1005Metric, F.Cu at (339.1, 108.6)
- added RCC2: 5.1k, Resistor_SMD:R_0402_1005Metric, F.Cu at (335.2, 110.5)
- added RRST1: 100k, acheron_Components:R_SMD_1026, F.Cu at (277.4, 155.1)
- added RSH1: 1M, acheron_Components:R_SMD_1026, F.Cu at (330.3, 102.8)
- added SW27: [{, acheron_MX:MX100H, F.Cu at (108.5, 127.6)
- added SW28: ]}, acheron_MX:MX150H, F.Cu at (84.7, 127.6)
- added SW43: Z, acheron_MX:MX100H, F.Cu at (303.7, 165.7)
- added SW44: X, acheron_MX:MX100H, F.Cu at (284.7, 165.7)
- added SW45: C, acheron_MX:MX100H, F.Cu at (265.6, 165.7)
- added SW46: V, acheron_MX:MX100H, F.Cu at (246.6, 165.7)
- added SW47: B, acheron_MX:MX100H, F.Cu at (227.5, 165.7)
- added SW48: N, acheron_MX:MX100H, F.Cu at (208.5, 165.7)
- added SW49: M, acheron_MX:MX100H, F.Cu at (189.4, 165.7)
- added SW50: <,, acheron_MX:MX100H, F.Cu at (170.4, 165.7)
- added SW51: .>, acheron_MX:MX100H, F.Cu at (151.3, 165.7)
- added SW52: ?/, acheron_MX:MX100H, F.Cu at (132.3, 165.7)
- added SWRST1: SW_Push, acheron_Hardware:smdPushBtn, F.Cu at (269.3, 154.9)
- added U1: STM32F072-LQFP48, acheron_Components:LQFP-48_7x7mm_P0.5mm, F.Cu at (326.3, 137.1)
- added U2: USBLC6-2SC6, acheron_Components:SOT-23-6, F.Cu at (336.6, 117.0)
- added U3: MCP1700-3302E_SOT23, Package_TO_SOT_SMD:SOT-23, F.Cu at (300.6, 115.5)
- SW1, SW10, SW11, SW12, SW13, SW16, SW17, SW18, SW19, SW2, SW20, SW21, SW22, SW23, SW3, SW30, SW31, SW32, SW33, SW34, SW35, SW36, SW37, SW38, SW4, SW5, SW6, SW7, SW8, SW9: footprint muente_plate:MX100 -> acheron_MX:MX100H; moved to F.Cu
- SW14: value BCKSPC_200 -> BKSP_200; footprint muente_plate:MX200 -> acheron_MX:MX200H; moved to F.Cu
- SW15: footprint muente_plate:MX100 -> acheron_MX:MX150H; moved to F.Cu
- SW24: value O -> L; footprint muente_plate:MX100 -> acheron_MX:MX100H; moved to F.Cu
- SW25: value P -> O; footprint muente_plate:MX100 -> acheron_MX:MX100H; moved to F.Cu
- SW26: value [{ -> P; footprint muente_plate:MX100 -> acheron_MX:MX100H; moved to F.Cu
- SW29: value CAPSLOCK_175 -> CAPS_175; footprint muente_plate:MX100 -> acheron_MX:MX175H; moved to F.Cu
- SW39: value ;: -> :;; footprint muente_plate:MX100 -> acheron_MX:MX100H; moved to F.Cu
- SW40: value ' -> "; footprint muente_plate:MX100 -> acheron_MX:MX100H; moved to F.Cu
- SW41: value ENTER_ISO -> ENTER_225; footprint muente_plate:MX200 -> acheron_MX:MX225H; moved to F.Cu
- SW42: value LSHIFT_125 -> LSHIFT_225; footprint muente_plate:MX100 -> acheron_MX:MX225H; moved to F.Cu
- SW53: footprint muente_plate:MX200 -> acheron_MX:MX275H; moved to F.Cu
- SW54: value LCTRL_125 -> MXSwitch; footprint muente_plate:MX100 -> acheron_MX:MX150H; moved to F.Cu
- SW55: value LGUI_125 -> MXSwitch; footprint muente_plate:MX100 -> acheron_MX:MX100H; moved to F.Cu
- SW56: value LALT_125 -> MXSwitch; footprint muente_plate:MX100 -> acheron_MX:MX150H; moved to F.Cu
- SW57: value SPACE_625 -> MXSwitch; footprint muente_plate:MX625 -> acheron_MX:MX700HR; moved to F.Cu
- SW58: value RALT_125 -> MXSwitch; footprint muente_plate:MX100 -> acheron_MX:MX150H; moved to F.Cu
- SW59: value RGUI_125 -> MXSwitch; footprint muente_plate:MX100 -> acheron_MX:MX100H; moved to F.Cu
- SW60: value FN_125 -> MXSwitch; footprint muente_plate:MX100 -> acheron_MX:MX150H; moved to F.Cu
- moved SW59 21.4 mm to (108.5, 184.7)
- moved SW60 21.4 mm to (84.7, 184.7)
- moved SW58 21.4 mm to (132.3, 184.7)
- moved SW41 13.5 mm to (91.8, 146.6), turned to 0 degrees
- moved SW57 11.9 mm to (213.2, 184.7)
- moved SW42 9.53 mm to (334.7, 165.7)
- moved SW54 2.38 mm to (341.8, 184.7)
- moved SW55 2.38 mm to (318.0, 184.7)
- moved SW56 2.38 mm to (294.2, 184.7)
- turned SW14 to 0 degrees
- turned SW53 to 0 degrees
Connections:
- SW1 pad 1: tierra -> Col1
- SW10 pad 1: tierra -> Col10
- SW11 pad 1: tierra -> Col11
- SW12 pad 1: tierra -> Col12
- SW13 pad 1: tierra -> Col13
- SW14 pad 1: tierra -> Col13
- SW15 pad 1: tierra -> Col1
- SW16 pad 1: tierra -> Col2
- SW17 pad 1: tierra -> Col3
- SW18 pad 1: tierra -> Col4
- SW19 pad 1: tierra -> Col5
- SW2 pad 1: tierra -> Col2
- SW20 pad 1: tierra -> Col6
- SW21 pad 1: tierra -> Col7
- SW22 pad 1: tierra -> Col8
- SW23 pad 1: tierra -> Col9
- SW24 pad 1: tierra -> Col10
- SW25 pad 1: tierra -> Col11
- SW26 pad 1: tierra -> Col12
- SW29 pad 1: tierra -> Col1
- SW3 pad 1: tierra -> Col3
- SW30 pad 1: tierra -> Col2
- SW31 pad 1: tierra -> Col3
- SW32 pad 1: tierra -> Col4
- SW33 pad 1: tierra -> Col5
- SW34 pad 1: tierra -> Col6
- SW35 pad 1: tierra -> Col7
- SW36 pad 1: tierra -> Col8
- SW37 pad 1: tierra -> Col9
- SW38 pad 1: tierra -> Col10
- SW39 pad 1: tierra -> Col11
- SW4 pad 1: tierra -> Col4
- SW41 pad 1: tierra -> Col13
- SW42 pad 1: tierra -> Col1
- SW5 pad 1: tierra -> Col5
- SW53 pad 1: tierra -> Col12
- SW54 pad 1: tierra -> Col1
- SW55 pad 1: tierra -> Col2
- SW56 pad 1: tierra -> Col3
- SW57 pad 1: tierra -> Col7
- SW58 pad 1: tierra -> Col10
- SW59 pad 1: tierra -> Col11
- SW6 pad 1: tierra -> Col6
- SW60 pad 1: tierra -> Col12
- SW7 pad 1: tierra -> Col7
- SW8 pad 1: tierra -> Col8
- SW9 pad 1: tierra -> Col9
Routing:
- net Row1: track 0.00 -> 481.5 mm
- net Row5: track 0.00 -> 481.3 mm
- net Col13: track 0.00 -> 366.5 mm
- net Row4: track 0.00 -> 356.5 mm
- net Col12: track 0.00 -> 328.1 mm, vias 0 -> 4
- net Col11: track 0.00 -> 305.9 mm, vias 0 -> 5
- net Row2: track 0.00 -> 304.9 mm
- net Col10: track 0.00 -> 270.1 mm, vias 0 -> 5
- net Row3: track 0.00 -> 269.2 mm, vias 0 -> 2
- net Col9: track 0.00 -> 224.6 mm, vias 0 -> 4
- net 3.3V: track 0.00 -> 211.1 mm, vias 0 -> 7
- net Col7: track 0.00 -> 208.2 mm, vias 0 -> 5
- net Col8: track 0.00 -> 199.5 mm, vias 0 -> 4
- net Col6: track 0.00 -> 162.5 mm, vias 0 -> 4
- net Col1: track 0.00 -> 158.7 mm, vias 0 -> 4
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- added copper zone on B.Cu, net /SHIELD
- added copper zone on B.Cu, net GND
- added copper zone on F.Cu, net GND
- removed copper zone on B.Cu, net tierra
- removed copper zone on F.Cu, net tierra
Other:
- board size 107 x 16 mm -> 283 x 94.2 mm
- board text added: "(I) If you want to check or reroute a specific trace, it is recommended that you use the High Contrast mode. Turn it on at View > Contrast mode > Check "High Contrast Mode". The icon is also available at the left icon column."
- board text added: "(II) It is recommended that the user has some knowledge in Git usage, since it is the main VCS tool used for the Acheron Project."
- board text added: "(III) All footprints are available either through KiCad's native libraries or the Acheron Library (http://github.com/Gondolindrim/AcheronLibrary). To facilitate the portability of the Acheron projects, this library is generally added at the ${KIPRJMOD} folder as a Git submodule. Hence, right after cloning the PCB repository, run: $ git submodule init --update To update the submodules."
- board text added: "(IV) For detailed information, check the Acheron Docs page for the KeebsPCB: http://gondolindrim.github.io/AcheronDocs/keebs/intro.html"
- board text added: "(i) The grid unit (1U) value used was 3/4" = 19.05mm"
- board text added: "(ii) The PCB was designed to fit the standards of the PCBWay manufacturer, at their cheapest settings."
- board text added: "(iii) All parts were quoted on the LCSC supplier (https://lcsc.com)."
- board text added: "(iv) You can always contact Gondolindrim through:"
- board text added: "(v) Most manufacturers list minimum character height as 0.8mm, and warn that any words using values below that will be undiscernable or unreadable. I have found that values down to 0.6mm (25 thou) can be used, although at that level a really close look is needed. Indeed, the minimum character height at which characters are easily readable is 0.8mm"
- board text added: "- Discord: Gondolindrim#9738"
- board text added: "- E-mail: alvaro.augusto.volpato@gmail.com"
- board text added: "- KeebsPCB's GitHub page: http://github.com/Gondolindrim/KeebsPCB"
- board text added: "- Reddit: /u/gondolindrim"
- board text added: "Also be sure to check with your parts supplier if they have all the necessary parts in the Bill of Materials and change parts and footprints accordingly to availability"
- board text added: "Be aware that capabilities may vary among manufacturers, so be sure to check with your manufacturer if they support the minimum values used."
- board text added: "GENERAL OBSERVATIONS"
- board text added: "GND"
- board text added: "MINIMUM CLEARANCE: 6 thou"
- board text added: "MINIMUM CLEARANCE: 8 thou"
- board text added: "MINIMUM VALUES"
- board text added: "NC"
- board text added: "PA0"
- board text added: "PA10"
- board text added: "PA5"
- board text added: "PA6"
- board text added: "PA7"
- board text added: "PA8"
- board text added: "PA9"
- board text added: "PB0"
- board text added: "PB1"
- board text added: "PB10"
- board text added: "PB11"
- board text added: "PB13"
- board text added: "PB14"
- board text added: "PB15"
- board text added: "PB2"
- board text added: "RECOMMENDED VALUES"
- board text added: "SILKSCREEN CHARACTER HEIGHT: 25 thou (see General Observation (v))"
- board text added: "SILKSCREEN CHARACTER HEIGHT: 32 thou"
- board text added: "SILKSCREEN CHARACTER TRACE WIDTH: 6 thou"
- board text added: "SILKSCREEN CHARACTER TRACE WIDTH: 8 thou"
- board text added: "TRACE WIDTH: 10 thou"
- board text added: "TRACE WIDTH: 6 thou (approx. 0.15 mm)"
- board text added: "TRACE-TO-EDGE AND VIA-TO-EDGE DISTANCE: 8 thou"
- board text added: "These are general hints to use this PCB file. They are aimed specially at thoise new to KiCad or ECAD in general and to whoever wishes to use this project."
- board text added: "These values were the default values used when possible."
- board text added: "USAGE GUIDE (PLEASE READ)"
- board text added: "VIA DIAMETER: 20 thou (approx. 0.5mm)"
- board text added: "VIA DIAMETER: 32 thou (approx. 0.8mm)"
- board text added: "VIA HOLE SIZE: 12 thou (approx. 0.3mm)"
- board text added: "VIA HOLE SIZE: 16 thou (approx. 0.4mm)"
- board text added: "VIA-TO-VIA AND VIA-TO-TRACE CLEARANCE: 6 thou"
- board text added: "VIA-TO-VIA AND VIA-TO-TRACE CLEARANCE: 8 thou"
