File: kicadFiles/keebsPCB.kicad_pcb (KiCad board)
At the start: 2 copper layers, 285.8 x 106.2 mm, 70 parts, among them SW1 ESC, SW10 9, SW11 0, SW12 -_, SW13 =+, SW14 BCKSPC_200, SW15 TAB_150, SW16 Q, SW17 W, SW18 E, SW19 R, SW2 1, SW20 T, SW21 Y, SW22 U, SW23 I, SW24 O, SW25 P, SW26 [{, SW27 ]}, SW28 KC_NUHS, SW29 CAPSLOCK_175, SW3 2, SW30 A, SW31 S, SW32 D, SW33 F, SW34 G, SW35 H, SW36 J, SW37 K, SW38 L, SW39 ;:, SW4 3, SW40 ', SW41 ENTER_ISO, SW42 LSHIFT_125, SW43 Z, SW44 X, SW45 C, SW46 V, SW47 B, SW48 N, SW49 M, SW5 4, SW50 ,<, SW51 .>, SW52 /?, SW53 RSHIFT_275, SW54 LCTRL_125, SW55 LGUI_125, SW56 LALT_125, SW57 SPACE_625, SW58 RALT_125, SW59 RGUI_125, SW6 5, SW60 FN_125, SW61 RCTRL_125, SW62 KC_NUBS, SW7 6, SW8 7, SW9 8

Commit message: rounded corners
Other:
- outline, holes or cut-outs redrawn
