File: kicadFiles/keebsPCB.sch (KiCad schematic (older format))
At the start: 165 parts, among them J1 TYPE-C-31-M12_13, J2 Conn_ARM_JTAG_SWD_10, J3 Conn_01x14, J4 Conn_01x14, SW1 ESC, SW10 9, SW11 0, SW12 -_, SW13 =+, SW14 BKSP_200, SW15 TAB_150, SW16 Q, SW17 W, SW18 E, SW19 R, SW2 1, SW20 T, SW21 Y, SW22 U, SW23 I, SW24 L, SW25 O, SW26 P, SW27 [{, SW28 ]}, SW29 CAPS_175, SW3 2, SW30 A, SW31 S, SW32 D, SW33 F, SW34 G, SW35 H, SW36 J, SW37 K, SW38 L, SW39 :;, SW4 3, SW40 \", SW41 ENTER_225, SW42 LSHIFT_225, SW43 Z, SW44 X, SW45 C, SW46 V, SW47 B, SW48 N, SW49 M, SW5 4, SW50 <,, SW51 .>, SW52 ?/, SW53 RSHIFT_275, SW54 MXSwitch, SW55 MXSwitch, SW56 MXSwitch, SW57 MXSwitch, SW58 MXSwitch, SW59 MXSwitch, SW6 5, SW60 MXSwitch, SW7 6, SW8 7, SW9 8, U1 STM32F072-LQFP48, U2 USBLC6-2SC6, U3 MCP1700-3302E_SOT23

Commit message: reset 2
Parts:
- removed D1, D10, D11, D12, D13, D14, D15, D16, D17, D18, D19, D2, D20, D21, D22, D23, D24, D25, D26, D27, D28, D29, D3, D30, D31, D32, D33, D34, D35, D36, D37, D38, D39, D4, D40, D41, D42, D43, D44, D45, D46, D47, D48, D49, D5, D50, D51, D52, D53, D54, D55, D56, D57, D58, D59, D6, D60, D7, D8, D9: 1N4148, acheron_Components:D_SOD-123, symbol Device:D
- removed H10, H8: Oval Mounting Hole, acheron_MountingHoles:MoutingHole_Oval_BackOnly_7mm_5.0x2.5mm, symbol Mechanical:MountingHole
- removed H7, H9: Oval Mounting Hole, acheron_MountingHoles:MoutingHole_Oval_7mm_5.0x2.5mm, symbol Mechanical:MountingHole
- removed J3: Conn_01x14, acheron_Connectors:PinHeader_1x7_P2.54mm_Vertical, symbol Connector_Generic:Conn_01x07
- removed J4: Conn_01x14, acheron_Connectors:PinHeader_1x8_P2.54mm_Vertical, symbol Connector_Generic:Conn_01x08
- removed L1: Keebs Logo, keebsLogo:keebsLogo, symbol Mechanical:MountingHole
- removed L2: OSHLogo, oshLogo:osh-logo, symbol Mechanical:MountingHole
- removed L3: Keebs Label, keebsLogo:keebsLabel, symbol Mechanical:MountingHole
- removed L4: Keebs Label Mask, keebsLogo:keebsLabelMask, symbol Mechanical:MountingHole
- added D1, D10, D11, D12, D13, D14, D15, D16, D17, D18, D19, D2, D20, D21, D22, D23, D24, D25, D26, D27, D28, D29, D3, D30, D31, D32, D33, D34, D35, D36, D37, D38, D39, D4, D40, D41, D42, D43, D44, D45, D46, D47, D48, D49, D5, D50, D51, D52, D53, D54, D55, D56, D57, D58, D59, D6, D60, D61, D62, D7, D8, D9: 1N4148, acheron_Components:D_SOD-123, symbol Device:D_Small
- added SW61: RCTRL_125, acheron_MX:MX125H, symbol acheronSymbols:MXSwitch
- added SW62: KC_NUBS, acheron_MX:MX100H, symbol acheronSymbols:MXSwitch
- SW14: value BKSP_200 -> BCKSPC_200
- SW24: value L -> O
- SW25: value O -> P
- SW26: value P -> [{
- SW27: value [{ -> ]}
- SW28: value ]} -> KC_NUHS; footprint acheron_MX:MX150H -> acheron_MX:MX100H
- SW29: value CAPS_175 -> CAPSLOCK_175
- SW39: value :; -> ;:
- SW40: value \" -> '\"
- SW41: value ENTER_225 -> ENTER_ISO; footprint acheron_MX:MX225H -> acheron_MX:MX_ISOEnter_Vertical
- SW42: value LSHIFT_225 -> LSHIFT_125; footprint acheron_MX:MX225H -> acheron_MX:MX125H
- SW50: value <, -> ,<
- SW52: value ?/ -> /?
- SW54: value MXSwitch -> LCTRL_125; footprint acheron_MX:MX150H -> acheron_MX:MX125H
- SW55: value MXSwitch -> LGUI_125; footprint acheron_MX:MX100H -> acheron_MX:MX125H
- SW56: value MXSwitch -> LALT_125; footprint acheron_MX:MX150H -> acheron_MX:MX125H
- SW57: value MXSwitch -> SPACE_625; footprint acheron_MX:MX700HR -> acheron_MX:MX625HR
- SW58: value MXSwitch -> RALT_125; footprint acheron_MX:MX150H -> acheron_MX:MX125H
- SW59: value MXSwitch -> RGUI_125; footprint acheron_MX:MX100H -> acheron_MX:MX125H
- SW60: value MXSwitch -> FN_125; footprint acheron_MX:MX150H -> acheron_MX:MX125H
Connections:
- net labels added: Col14
- net labels removed: Extra1, Extra10, Extra11, Extra12, Extra13, Extra14, Extra15, Extra2, Extra3, Extra4, Extra5, Extra6, Extra7, Extra8, Extra9
- wire segments 348 -> 338
Other:
- note removed: "Extra pins"
- note removed: "Logos and flags"
- note removed: "Switch matrix"

Commit message: remade plate
Parts:
- removed CB1: 1uF, Capacitor_SMD:C_0402_1005Metric, symbol Device:C_Small
- removed CB2: 10n, Capacitor_SMD:C_0402_1005Metric, symbol Device:C_Small
- removed CB3, CB5, CB8, CUSB1: 100n, Capacitor_SMD:C_0402_1005Metric, symbol Device:C_Small
- removed CB4, CB6: 4.7uF, Capacitor_SMD:C_0402_1005Metric, symbol Device:C_Small
- removed CB7: 100nF, Capacitor_SMD:C_0402_1005Metric, symbol Device:C_Small
- removed CRST1, CSI1: 10u, Capacitor_SMD:C_0805_2012Metric_Pad1.15x1.40mm_HandSolder, symbol Device:C_Small
- removed CRST2: 4.7n, Capacitor_SMD:C_0805_2012Metric_Pad1.15x1.40mm_HandSolder, symbol Device:C_Small
- removed CSH1: 4.7nF, Capacitor_SMD:C_0805_2012Metric, symbol Device:C_Small
- removed CSO1: 1u, Capacitor_SMD:C_0805_2012Metric_Pad1.15x1.40mm_HandSolder, symbol Device:C_Small
- removed D1, D10, D11, D12, D13, D14, D15, D16, D17, D18, D19, D2, D20, D21, D22, D23, D24, D25, D26, D27, D28, D29, D3, D30, D31, D32, D33, D34, D35, D36, D37, D38, D39, D4, D40, D41, D42, D43, D44, D45, D46, D47, D48, D49, D5, D50, D51, D52, D53, D54, D55, D56, D57, D58, D59, D6, D60, D61, D62, D7, D8, D9: 1N4148, acheron_Components:D_SOD-123, symbol Device:D_Small
- removed DF1: RB060M-60TR, acheron_Components:D_SOD-123, symbol Device:D_Schottky
- removed DRST1, DS1: 1N4148, acheron_Components:D_SOD-123, symbol Device:D
- removed F1: Polyfuse, acheron_Components:Fuse_1812_4532, symbol Device:Polyfuse_Small
- removed H1, H6: Half Side Hole, acheron_MountingHoles:halfSideHole, symbol Mechanical:MountingHole
- removed H2: Mounting Hole, acheron_MountingHoles:MoutingHole_Oval_7mm_5.0x2.5mm, symbol Mechanical:MountingHole
- removed H3, H5: Oval Mounting Hole, acheron_MountingHoles:MoutingHole_Oval_BackOnly_7mm_5.0x2.5mm, symbol Mechanical:MountingHole
- removed H4: Oval Mounting Hole, acheron_MountingHoles:MoutingHole_Oval_7mm_5.0x2.5mm, symbol Mechanical:MountingHole
- removed J1: TYPE-C-31-M12_13, acheron_Connectors:TYPE-C-31-M-12, symbol acheronSymbols:TYPE-C-31-M12_13
- removed J2: Conn_ARM_JTAG_SWD_10, acheron_Connectors:Conn_ARM_JTAG_SWD_10, symbol Connector:Conn_ARM_JTAG_SWD_10
- removed QRST1: DTC123J, Package_TO_SOT_SMD:SOT-23, symbol Transistor_BJT:DTC123J
- removed RCC1, RCC2: 5.1k, Resistor_SMD:R_0402_1005Metric, symbol Device:R_Small
- removed RRST1: 100k, acheron_Components:R_SMD_1026, symbol Device:R_Small
- removed RSH1: 1M, acheron_Components:R_SMD_1026, symbol Device:R_Small
- removed SWRST1: SW_Push, acheron_Hardware:smdPushBtn, symbol Switch:SW_Push
- removed U1: STM32F072-LQFP48, acheron_Components:LQFP-48_7x7mm_P0.5mm, symbol acheronSymbols:STM32F072-LQFP48
- removed U2: USBLC6-2SC6, acheron_Components:SOT-23-6, symbol Power_Protection:USBLC6-2SC6
- removed U3: MCP1700-3302E_SOT23, Package_TO_SOT_SMD:SOT-23, symbol Regulator_Linear:MCP1700-3302E_SOT23
- SW1, SW10, SW11, SW12, SW13, SW16, SW17, SW18, SW19, SW2, SW20, SW21, SW22, SW23, SW24, SW25, SW26, SW27, SW28, SW3, SW30, SW31, SW32, SW33, SW34, SW35, SW36, SW37, SW38, SW39, SW4, SW40, SW43, SW44, SW45, SW46, SW47, SW48, SW49, SW5, SW50, SW51, SW52, SW6, SW62, SW7, SW8, SW9: footprint acheron_MX:MX100H -> muente_plate:MX100
- SW14: footprint acheron_MX:MX200H -> muente_plate:MX200
- SW15: footprint acheron_MX:MX150H -> muente_plate:MX100
- SW29: footprint acheron_MX:MX175H -> muente_plate:MX100
- SW41: footprint acheron_MX:MX_ISOEnter_Vertical -> muente_plate:MX200
- SW42, SW54, SW55, SW56, SW58, SW59, SW60, SW61: footprint acheron_MX:MX125H -> muente_plate:MX100
- SW53: footprint acheron_MX:MX275H -> muente_plate:MX200
- SW57: footprint acheron_MX:MX625HR -> muente_plate:MX625
Connections:
- net labels added: tierra
- net labels removed: 3.3V, 5V, BOOT0, Col1, Col10, Col11, Col12, Col13, Col14, Col2, Col3, Col4, Col5, Col6, Col7, Col8, Col9, D+, D-, DBus+, DBus-, GND, NRST, Row1, Row2, Row3, Row4, Row5, SHIELD, SWCLK, SWDIO, VBUS
- wire segments 338 -> 151
- no-connect marks 4 -> 0
Other:
- note removed: "CBx are the bypass capacitors. Their value is specified in reference [2]."
- note removed: "Hard reset circuit"
- note removed: "MCU"
- note removed: "Mounting holes"
- note removed: "Power supply and protection circuit"
- note removed: "SWD"
- note removed: "Shield"
- note removed: "USB Connector"
- note removed: "USD ESD"
